Commit message: removes world joint fixed link from urdf models

File: ur_description/urdf/ur10_joint_limited_robot.urdf.xacro (robot description, xacro)
@@ -19,9 +19,3 @@
     kinematics_file="${load_yaml('$(arg kinematics_config)')}"
 />
-  <link name="world" />
-  <joint name="world_joint" type="fixed">
-    <parent link="world" />
-    <child link = "base_link" />
-    <origin xyz="0.0 0.0 0.0" rpy="0.0 0.0 0.0" />
-  </joint>
 </robot>

File: ur_description/urdf/ur10_robot.urdf.xacro (robot description, xacro)
@@ -13,9 +13,3 @@
     kinematics_file="${load_yaml('$(arg kinematics_config)')}"
   />
-  <link name="world" />
-  <joint name="world_joint" type="fixed">
-    <parent link="world" />
-    <child link = "base_link" />
-    <origin xyz="0.0 0.0 0.0" rpy="0.0 0.0 0.0" />
-  </joint>
 </robot>
